File: ScoutMakes FM Kit/ScoutMakes_FM_Kit.brd (EAGLE design)
At the start: 50.9 x 39.1 mm, 20 parts, among them J1 35RASMT2BHNTRX, Q2 BSS138BKS, U1 TEA5767, U2 AP2112K-3.3

Commit message: Updated board files
Parts:
- removed C1: 0.1uF, microbuilder:0603-NO
- removed C2: 10uF, microbuilder:0805-NO
- removed CONN4: SM04B-SRSS-TB, microbuilder:JST_SH4
- removed D3: RED, microbuilder:CHIPLED_0805_NOOUTLINE
- removed D5: MBR120, microbuilder:SOD-123
- removed J1: 35RASMT2BHNTRX, 35RASMT2BHNTRX_3point5mm:SWITCHCRAFT_35RASMT2BHNTRX
- removed Q2: BSS138BKS, microbuilder:SOT363
- removed RN1: CAY16-103J4LF, CAY16-103J4LF:RESCAF80P320X160X60-8N
- removed U2: AP2112K-3.3, microbuilder:SOT23-5
- added C11, C12: 4.7nF, microbuilder:0805-NO
- added C4: 10uF, microbuilder:0805-NO
- added J2: SJ-43514-SMT, SJ-43514-SMT:CUI_SJ-43514-SMT
- added R2: 10K, microbuilder:0603-NO
- added R3, R6: 470, microbuilder:0805-NO
- moved C3 9.20 mm to (36.8, 22.9)
- moved R1 5.28 mm to (27.2, 31.9), turned to 0 degrees
- moved U1 0.29 mm to (20.4, 24.4)
- moved ANT 0.27 mm to (1.78, 23.9)
Connections:
- removed net 3V: D5.A, MS2.2
- removed net LOUT: J1.4, U1.7
- removed net N$1: D3.A, R1.2
- removed net ROUT: J1.1, U1.8
- removed net SCL_3V: MS2.18, Q2.1, RN1.3, U1.2
- removed net SDA_3V: MS2.17, Q2.4, RN1.4, U1.1
- removed net VCC: C2.1, CONN4.2, RN1.7, RN1.8, U2.1, U2.3
- new net L_AC: C3.1, J2.2
- new net L_OUT: R3.1, U1.7
- new net N$5: C12.1, C4.2, R6.2
- new net N$6: C11.1, C3.2, R3.2
- new net R_AC: C4.1, J2.3
- new net R_OUT: R6.1, U1.8
- net 3.3V: now also MS2.2, R2.1; no longer C1.1, C3.1, D5.C, Q2.2, Q2.5, RN1.5, RN1.6, U2.5
- net GND: now also C11.2, C12.2, J2.1, J2.4; no longer C1.2, C2.2, C3.2, CONN4.1, D3.C, J1.5, U2.2
- net SCL: now also MS2.18, R1.2, U1.2; no longer CONN4.4, Q2.6, RN1.1
- net SDA: now also MS2.17, R2.2, U1.1; no longer CONN4.3, Q2.3, RN1.2
Routing:
- net VCC: track 44.2 -> 0.00 mm, vias 2 -> 0
- net SDA_3V: track 38.9 -> 0.00 mm, vias 2 -> 0
- net ROUT: track 38.5 -> 0.00 mm, vias 2 -> 0
- net SCL_3V: track 37.1 -> 0.00 mm, vias 2 -> 0
- net N$1: track 36.4 -> 0.00 mm, vias 2 -> 0
- net R_OUT: track 0.00 -> 35.7 mm
- net LOUT: track 32.8 -> 0.00 mm
- net 3.3V: track 36.5 -> 5.85 mm, vias 0 -> 1
- net 3V: track 23.0 -> 0.00 mm, vias 1 -> 0
- net GND: track 0.00 -> 21.0 mm, vias 0 -> 2
- net L_OUT: track 0.00 -> 20.6 mm, vias 0 -> 2
- net ANT: track 7.47 -> 27.9 mm
- net SDA: track 30.4 -> 47.8 mm, vias 4 -> 0
- net N$6: track 0.00 -> 16.9 mm
- net R_AC: track 0.00 -> 15.0 mm
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Other:
- board text removed: "PWR"
