File: ScoutMakes FM Kit/ScoutMakes_FM_Kit.sch (EAGLE design)
At the start: 20 parts, among them J1 35RASMT2BHNTRX, Q2 BSS138BKS, U1 TEA5767, U2 AP2112K-3.3

Commit message: Updated board files
Parts:
- removed C1: 0.1uF, microbuilder:CAP_CERAMIC0603_NO
- removed C2: 10uF, microbuilder:CAP_CERAMIC0805-NOOUTLINE
- removed CONN4: SM04B-SRSS-TB, microbuilder:STEMMA_I2C_QT
- removed D3: RED, microbuilder:LED0805_NOOUTLINE
- removed D5: MBR120, microbuilder:DIODE-SCHOTTKYSOD-123
- removed J1: 35RASMT2BHNTRX, 35RASMT2BHNTRX_3point5mm:35RASMT2BHNTRX
- removed Q2: BSS138BKS, microbuilder:MOSFET-N_DUAL
- removed RN1: CAY16-103J4LF, CAY16-103J4LF:CAY16-103J4LF
- removed U2: AP2112K-3.3, microbuilder:VREG_SOT23-5
- added C11, C12: 4.7nF, microbuilder:CAP_CERAMIC0805-NOOUTLINE
- added C4: 10uF, microbuilder:CAP_CERAMIC0805-NOOUTLINE
- added J2: SJ-43514-SMT, SJ-43514-SMT:SJ-43514-SMT
- added R2: 10K, microbuilder:RESISTOR_0603_NOOUT
- added R3, R6: 470, microbuilder:RESISTOR0805_NOOUTLINE
Connections:
- removed net 3V: D5.A, MS2.3V
- removed net LOUT: J1.4, U1.7.LOUT
- removed net N$1: D3.A, R1.2
- removed net ROUT: J1.1, U1.8.ROUT
- removed net SCL_3V: MS2.GPIOSCL, Q21.S, RN1.3, U1.2.CLK
- removed net SDA_3V: MS2.GPIOSDA, Q22.S, RN1.4, U1.1.DATA
- removed net VCC: C2.1, CONN4G$1.V+, RN1.7, RN1.8, U2.EN, U2.IN
- new net L_AC: C3.1, J2.TIP
- new net L_OUT: R3.1, U1.7.LOUT
- new net N$5: C12.1, C4.2, R6.2
- new net N$6: C11.1, C3.2, R3.2
- new net R_AC: C4.1, J2.RING1
- new net R_OUT: R6.1, U1.8.ROUT
- net 3.3V: now also MS2.3V, R2.1; no longer C1.1, C3.1, D5.C, Q21.G, Q22.G, RN1.5, RN1.6, U2.OUT
- net GND: now also C11.2, C12.2, J2.RING2, J2.SLEEVE; no longer C1.2, C2.2, C3.2, CONN4G$1.GND, D3.C, J1.5, U2.GND
- net SCL: now also MS2.GPIOSCL, R1.2, U1.2.CLK; no longer CONN4G$1.SCL, Q21.D, RN1.1
- net SDA: now also MS2.GPIOSDA, R2.2, U1.1.DATA; no longer CONN4G$1.SDA, Q22.D, RN1.2
Other:
- note added: "10/23/2020"
- note added: "4"
- note added: "PUSH BUTTONS"
- note added: "SCOUTMAKES FM RADIO EXPANSION BOARD"
- note added: "TinkeringTech"
- note removed: "D"
- note removed: "G"
- note removed: "I2C Pullups & Shift"
- note removed: "ON LED"
- note removed: "Power supply"
- note removed: "S"
- note removed: "STEMMA/I2C Headers"
- moved on the sheet: ANT, C3, R1, S1, S2, S3, S4, S5, S6
